File: testProj/breakout-pcb's/breakout_pwr/breakout_pwr.kicad_pcb (KiCad board)
At the start: 2 copper layers, 45.5 x 30 mm, 33 parts, among them J1 Conn_01x05, J2 Conn_02x05_Odd_Even, J3 Screw_Terminal_01x05, U1 LM1117DT-5.0, U2 ADP150AUJZ-3.3-R7

Commit message: in prog schematics
Other:
- board text removed: "<3 WZL-kun <3"
Changed lines of the file:
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@@
-		)
-	)
-	(gr_text "<3 WZL-kun <3"
-		(at 173 56 -90)
-		(layer "B.SilkS")
-		(effects
-			(font
-				(size 1 1)
-				(thickness 0.1)
-			)
-			(justify left bottom mirror)
 		)
 	)
